Commit message: Updated robotarm_moveit_config

File: robotarm_moveit_config/config/robotarm1.ros2_control.xacro (robot description, xacro)
@@ -1,5 +1,5 @@
 <?xml version="1.0"?>
 <robot xmlns:xacro="http://www.ros.org/wiki/xacro">
-    <xacro:macro name="cocoabot_ros2_control" params="name initial_positions_file">
+    <xacro:macro name="robotarm1_ros2_control" params="name initial_positions_file">
         <xacro:property name="initial_positions" value="${load_yaml(initial_positions_file)['initial_positions']}"/>
         <ros2_control name="${name}" type="system">
@@ -8,4 +8,11 @@
                 <plugin>mock_components/GenericSystem</plugin>
             </hardware>
+            <joint name="joint_7">
+                <command_interface name="position"/>
+                <state_interface name="position">
+                  <param name="initial_value">${initial_positions['joint_7']}</param>
+                </state_interface>
+                <state_interface name="velocity"/>
+            </joint>
             <joint name="joint_1">
                 <command_interface name="position"/>
@@ -43,8 +50,8 @@
                 <state_interface name="velocity"/>
             </joint>
-            <joint name="right_gripper_joint">
+            <joint name="tcp_joint">
                 <command_interface name="position"/>
                 <state_interface name="position">
-                  <param name="initial_value">${initial_positions['right_gripper_joint']}</param>
+                  <param name="initial_value">${initial_positions['tcp_joint']}</param>
                 </state_interface>
                 <state_interface name="velocity"/>
