Commit message: new moveit config

File: robotarm_moveit_config/config/robotarm.ros2_control.xacro (robot description, xacro)
@@ -1,5 +1,5 @@
 <?xml version="1.0"?>
 <robot xmlns:xacro="http://www.ros.org/wiki/xacro">
-    <xacro:macro name="robotarm1_ros2_control" params="name initial_positions_file">
+    <xacro:macro name="robotarm_ros2_control" params="name initial_positions_file">
         <xacro:property name="initial_positions" value="${load_yaml(initial_positions_file)['initial_positions']}"/>
         <ros2_control name="${name}" type="system">
@@ -8,11 +8,4 @@
                 <plugin>mock_components/GenericSystem</plugin>
             </hardware>
-            <joint name="joint_7">
-                <command_interface name="position"/>
-                <state_interface name="position">
-                  <param name="initial_value">${initial_positions['joint_7']}</param>
-                </state_interface>
-                <state_interface name="velocity"/>
-            </joint>
             <joint name="joint_1">
                 <command_interface name="position"/>
@@ -57,4 +50,11 @@
                 <state_interface name="velocity"/>
             </joint>
+            <joint name="joint_7">
+                <command_interface name="position"/>
+                <state_interface name="position">
+                  <param name="initial_value">${initial_positions['joint_7']}</param>
+                </state_interface>
+                <state_interface name="velocity"/>
+            </joint>
         </ros2_control>
     </xacro:macro>

File: robotarm_moveit_config/config/robotarm.urdf.xacro (robot description, xacro)
@@ -1,9 +1,9 @@
 <?xml version="1.0"?>
-<robot xmlns:xacro="http://www.ros.org/wiki/xacro" name="robotarm1">
+<robot xmlns:xacro="http://www.ros.org/wiki/xacro" name="robotarm">
     <xacro:arg name="initial_positions_file" default="initial_positions.yaml" />
-    <!-- Import robotarm1 urdf file -->
+    <!-- Import robotarm urdf file -->
     <xacro:include filename="$(find robotarm_description)/urdf/robotarm.urdf" />
     <!-- Import control_xacro -->
-    <xacro:include filename="robotarm1.ros2_control.xacro" />
-    <xacro:robotarm1_ros2_control name="FakeSystem" initial_positions_file="$(arg initial_positions_file)"/>
+    <xacro:include filename="robotarm.ros2_control.xacro" />
+    <xacro:robotarm_ros2_control name="FakeSystem" initial_positions_file="$(arg initial_positions_file)"/>
 </robot>
