Commit message: Updated robotarm_description

File: robotarm_description/urdf/final_arm.urdf (robot description, URDF)
Before this commit: robot cocoabot, 12 links, 11 joints
Links:
- removed link camera_link
- removed link left_cutter_link
- removed link left_gripper_link
- removed link right_cutter_link
- removed link right_gripper_link
- added link link_6, mass 0.011608; collision mesh filename=package://robotarm_description/meshes/link_6.STL; visual mesh filename=package://robotarm_description/meshes/link_6.STL
- added link link_7, mass 0.011608; collision mesh filename=package://robotarm_description/meshes/link_7.STL; visual mesh filename=package://robotarm_description/meshes/link_7.STL
- link base_link: mass 0.15177 -> 0.4726
- link link_1: mass 0.19298 -> 0.25582
- link link_2: mass 0.34787 -> 0.2619
- link link_3: mass 0.24803 -> 0.23372
- link link_4: mass 0.13001 -> 0.11094
- link link_5: mass 0.35342 -> 0.15528
Joints:
- removed joint camera_joint
- removed joint left_cutter_joint
- removed joint left_gripper_joint
- removed joint right_cutter_joint
- removed joint right_gripper_joint
- added joint joint_6: type prismatic, parent link_5, child link_6, origin xyz=0.075 0 -0.02 rpy=0 0 0, axis 0 1 0, limit lower=0 upper=0.04 effort=3.34 velocity=1, mimic joint=joint_7 multiplier=-1 offset=0
- added joint joint_7: type prismatic, parent link_5, child link_7, origin xyz=0.075 0 -0.02 rpy=0 0 0, axis 0 1 0, limit lower=-0.04 upper=0 effort=3.34 velocity=1
- joint joint_1: axis 0 0 1 -> 0 0 -1; limit lower=-1.57 upper=1.57 effort=8.33 velocity=1 -> lower=-1.571 upper=1.571 effort=8.33 velocity=1; origin xyz=0 0 0.0627 rpy=0 0 0 -> xyz=0 0 0.0617 rpy=0 0 0
- joint joint_2: limit lower=0 upper=3.142 effort=16.67 velocity=1 -> lower=0.0 upper=3.142 effort=15.7 velocity=1; origin xyz=0 0 0.058 rpy=0 0 0 -> xyz=-0.0002 0.03525 0.0605 rpy=0 0 0
- joint joint_3: axis -1 0 0 -> 0 -1 0; limit lower=-3.142 upper=0 effort=16.67 velocity=1 -> lower=0 upper=3.142 effort=15.7 velocity=1; origin xyz=-0.291 0 0 rpy=1.5708 0 -1.5708 -> xyz=-0.26 -0.00065 -0.00065 rpy=0 0 0
- joint joint_4: axis 0 -1 0 -> 0 1 0; limit lower=-1.57 upper=1.57 effort=8.33 velocity=1 -> lower=-1.571 upper=1.571 effort=8.34 velocity=1; origin xyz=5E-05 0.043049 -0.29 rpy=-1.5708 1.5708 0 -> xyz=0.2602 -0.00325 0.046162 rpy=0 0 0
- joint joint_5: limit lower=-1.57 upper=1.57 effort=8.33 velocity=1 -> lower=-1.571 upper=1.571 effort=8.34 velocity=1; origin xyz=0.0947 -1.9981E-05 -5.0149E-05 rpy=0 0 0 -> xyz=0.0947 -0.03305 0.0003 rpy=0 0 0
- joint tcp_joint: origin xyz=0.125 0 -0.03 rpy=0 0 0 -> xyz=0.12 0 0 rpy=0 0 0
