Commit message: Chages on robotarm meshes

File: robotarm_description/urdf/robotarm.urdf (robot description, URDF)
Before this commit: robot robotarm1, 9 links, 8 joints
Links:
- link base_link: mass 0.4726 -> 0.49164
- link link_1: mass 0.25582 -> 0.25792
- link link_2: mass 0.2619 -> 0.26072
- link link_3: mass 0.23372 -> 0.24699
- link link_4: mass 0.11094 -> 0.13001
- link link_5: mass 0.15528 -> 0.14243
- link link_6: mass 0.011608 -> 0.012327
- link link_7: mass 0.011608 -> 0.012327
Joints:
- joint joint_1: origin xyz=0 0 0.0617 rpy=0 0 0 -> xyz=0 0 0.0632 rpy=0 0 0
- joint joint_2: limit lower=0.0 upper=3.142 effort=15.7 velocity=1 -> lower=0 upper=3.142 effort=15.7 velocity=1; origin xyz=-0.0002 0.03525 0.0605 rpy=0 0 0 -> xyz=0.0002 0.03575 0.062 rpy=0 0 0
- joint joint_3: origin xyz=-0.26 -0.00065 -0.00065 rpy=0 0 0 -> xyz=-0.26 5E-05 -0.00025 rpy=0 0 0
- joint joint_4: origin xyz=0.2602 -0.00325 0.046162 rpy=0 0 0 -> xyz=0.2602 -0.00245 0.046362 rpy=0 0 0
- joint joint_5: origin xyz=0.0947 -0.03305 0.0003 rpy=0 0 0 -> xyz=0.0947 -0.03245 -0.0003 rpy=0 0 0
- joint joint_6: origin xyz=0.075 0 -0.02 rpy=0 0 0 -> xyz=0.072 0 -0.02 rpy=0 0 0
- joint joint_7: origin xyz=0.075 0 -0.02 rpy=0 0 0 -> xyz=0.072 0 -0.02 rpy=0 0 0
